Commit message: Change dimensions to MiR250

File: description/gazebo_control.xacro (robot description, xacro)
@@ -6,8 +6,8 @@
             <left_joint>left_wheel_joint</left_joint>
             <right_joint>right_wheel_joint</right_joint>
-            <wheel_separation>0.35</wheel_separation>
+            <wheel_separation>0.63</wheel_separation>
             <wheel_radius>0.05</wheel_radius>
             <!-- Limits -->
-            <max_linear_acceleration>0.33</max_linear_acceleration>
+            <max_linear_acceleration>0.66</max_linear_acceleration>
             <!-- Input -->
             <topic>/cmd_vel</topic>
@@ -16,5 +16,5 @@
             <child_frame_id>base_link</child_frame_id>
             <odom_topic>/odom</odom_topic>
-            <odom_publisher_frequency>30</odom_publisher_frequency>
+            <odom_publisher_frequency>100</odom_publisher_frequency>
             <tf_topic>/tf</tf_topic>
         </plugin>

File: description/robot.urdf.xacro (robot description, xacro)
@@ -6,8 +6,8 @@
             <left_joint>left_wheel_joint</left_joint>
             <right_joint>right_wheel_joint</right_joint>
-            <wheel_separation>0.35</wheel_separation>
+            <wheel_separation>0.63</wheel_separation>
             <wheel_radius>0.05</wheel_radius>
             <!-- Limits -->
-            <max_linear_acceleration>0.33</max_linear_acceleration>
+            <max_linear_acceleration>0.66</max_linear_acceleration>
             <!-- Input -->
             <topic>/cmd_vel</topic>
@@ -16,5 +16,5 @@
             <child_frame_id>base_link</child_frame_id>
             <odom_topic>/odom</odom_topic>
-            <odom_publisher_frequency>30</odom_publisher_frequency>
+            <odom_publisher_frequency>100</odom_publisher_frequency>
             <tf_topic>/tf</tf_topic>
         </plugin>

File: description/robot_core.xacro (robot description, xacro)
@@ -14,22 +14,22 @@
         <parent link="base_link"/>
         <child link="chassis"/>
-        <origin xyz="-0.1 0 0"/>
+        <origin xyz="0 0 0"/>
     </joint>
     <link name="chassis">
         <visual>
-            <origin xyz="0.15 0 0.075" rpy="0 0 0"/>
+            <origin xyz="0 0 0.15" rpy="0 0 0"/>
             <geometry>
-                <box size="0.3 0.3 0.15"/>
+                <box size="0.8 0.58 0.3"/>
             </geometry>
             <material name="white"/>
         </visual>
         <collision>
-            <origin xyz="0.15 0 0.075" rpy="0 0 0"/>
+            <origin xyz="0 0 0.15" rpy="0 0 0"/>
             <geometry>
-                <box size="0.3 0.3 0.15"/>
+                <box size="0.8 0.58 0.3"/>
             </geometry>
         </collision>
-        <xacro:inertial_box mass="0.5" x="0.3" y="0.3" z="0.15">
-            <origin xyz="0.15 0 0.075" rpy="0 0 0"/>
+       <xacro:inertial_box mass="84" x="0.8" y="0.58" z="0.3">
+            <origin xyz="0 0 0.15" rpy="0 0 0"/>
         </xacro:inertial_box>
     </link>
@@ -38,5 +38,5 @@
         <parent link="base_link"/>
         <child link="left_wheel"/>
-        <origin xyz="0 0.175 0" rpy="-${pi/2} 0 0"/>
+        <origin xyz="0 0.31 0" rpy="-${pi/2} 0 0"/>
         <axis xyz="0 0 1"/>
     </joint>
@@ -53,5 +53,5 @@
             </geometry>
         </collision>
-        <xacro:inertial_cylinder mass="0.1" length="0.04" radius="0.05">
+        <xacro:inertial_cylinder mass="1" length="0.04" radius="0.05">
             <origin xyz="0 0 0" rpy="0 0 0"/>
         </xacro:inertial_cylinder>
@@ -61,5 +61,5 @@
         <parent link="base_link"/>
         <child link="right_wheel"/>
-        <origin xyz="0 -0.175 0" rpy="${pi/2} 0 0"/>
+        <origin xyz="0 -0.31 0" rpy="${pi/2} 0 0"/>
         <axis xyz="0 0 -1"/>
     </joint>
@@ -76,15 +76,15 @@
             </geometry>
         </collision>
-        <xacro:inertial_cylinder mass="0.1" length="0.04" radius="0.05">
+        <xacro:inertial_cylinder mass="1" length="0.04" radius="0.05">
             <origin xyz="0 0 0" rpy="0 0 0"/>
         </xacro:inertial_cylinder>
     </link>
-    <!-- Caster Wheel -->
-    <joint name="caster_wheel_joint" type="fixed">
+    <!-- Caster Wheels -->
+    <joint name="top_left_caster_wheel_joint" type="fixed">
         <parent link="chassis"/>
-        <child link="caster_wheel"/>
-        <origin xyz="0.24 0 0" rpy="0 0 0"/>
+        <child link="top_left_caster_wheel"/>
+        <origin xyz="0.34 0.235 0" rpy="0 0 0"/>
     </joint>
-    <link name="caster_wheel">
+    <link name="top_left_caster_wheel">
         <visual>
             <geometry>
@@ -98,9 +98,84 @@
             </geometry>
         </collision>
-        <xacro:inertial_sphere mass="0.1" radius="0.05">
+        <xacro:inertial_sphere mass="2" radius="0.05">
             <origin xyz="0 0 0" rpy="0 0 0"/>
         </xacro:inertial_sphere>
     </link>
-    <gazebo reference="caster_wheel">
+    <gazebo reference="top_left_caster_wheel">
+        <mu1 value="0.001" />
+        <mu2 value="0.001" />
+    </gazebo>
+    <joint name="top_right_caster_wheel_joint" type="fixed">
+        <parent link="chassis"/>
+        <child link="top_right_caster_wheel"/>
+        <origin xyz="0.34 -0.235 0" rpy="0 0 0"/>
+    </joint>
+    <link name="top_right_caster_wheel">
+        <visual>
+            <geometry>
+                <sphere radius="0.05"/>
+            </geometry>
+            <material name="black"/>
+        </visual>
+        <collision>
+            <geometry>
+                <sphere radius="0.05"/>
+            </geometry>
+        </collision>
+        <xacro:inertial_sphere mass="2" radius="0.05">
+            <origin xyz="0 0 0" rpy="0 0 0"/>
+        </xacro:inertial_sphere>
+    </link>
+    <gazebo reference="top_right_caster_wheel">
+        <mu1 value="0.001" />
+        <mu2 value="0.001" />
+    </gazebo>
+    <joint name="bottom_left_caster_wheel_joint" type="fixed">
+        <parent link="chassis"/>
+        <child link="bottom_left_caster_wheel"/>
+        <origin xyz="-0.34 0.235 0" rpy="0 0 0"/>
+    </joint>
+    <link name="bottom_left_caster_wheel">
+        <visual>
+            <geometry>
+                <sphere radius="0.05"/>
+            </geometry>
+            <material name="black"/>
+        </visual>
+        <collision>
+            <geometry>
+                <sphere radius="0.05"/>
+            </geometry>
+        </collision>
+        <xacro:inertial_sphere mass="2" radius="0.05">
+            <origin xyz="0 0 0" rpy="0 0 0"/>
+        </xacro:inertial_sphere>
+    </link>
+    <gazebo reference="bottom_left_caster_wheel">
+        <mu1 value="0.001" />
+        <mu2 value="0.001" />
+    </gazebo>
+    <joint name="bottom_right_caster_wheel_joint" type="fixed">
+        <parent link="chassis"/>
+        <child link="bottom_right_caster_wheel"/>
+        <origin xyz="-0.34 -0.235 0" rpy="0 0 0"/>
+    </joint>
+    <link name="bottom_right_caster_wheel">
+        <visual>
+            <geometry>
+                <sphere radius="0.05"/>
+            </geometry>
+            <material name="black"/>
+        </visual>
+        <collision>
+            <geometry>
+                <sphere radius="0.05"/>
+            </geometry>
+        </collision>
+        <xacro:inertial_sphere mass="2" radius="0.05">
+            <origin xyz="0 0 0" rpy="0 0 0"/>
+        </xacro:inertial_sphere>
+    </link>
+    <gazebo reference="bottom_right_caster_wheel">
         <mu1 value="0.001" />
         <mu2 value="0.001" />
