Commit message: Attach arm to platform

File: description/robot_core.xacro (robot description, xacro)
@@ -181,3 +181,5 @@
         <mu2 value="0.001" />
     </gazebo>
+    <!-- Include Arm URDF -->
+    <xacro:include filename="$(find my_ur)/urdf/ur.urdf.xacro" />
 </robot>

File: description/ros2_control.xacro (robot description, xacro)
@@ -6,4 +6,5 @@
             <plugin>gz_ros2_control/GazeboSimSystem</plugin>
         </hardware>
+        <!-- Platform Joints -->
         <joint name="left_wheel_joint">
             <command_interface name="velocity">
@@ -22,4 +23,126 @@
             <state_interface name="velocity"/>
         </joint>
+        <!-- Arm joints -->
+        <joint name="shoulder_pan_joint">
+            <command_interface name="position"/>
+            <command_interface name="velocity"/>
+            <state_interface name="position">
+                <param name="initial_value">0</param>
+            </state_interface>
+            <state_interface name="velocity"/>
+            <state_interface name="effort"/>
+        </joint>
+        <joint name="shoulder_lift_joint">
+            <command_interface name="position"/>
+            <command_interface name="velocity"/>
+            <state_interface name="position">
+                <param name="initial_value">-1.57</param>
+            </state_interface>
+            <state_interface name="velocity"/>
+            <state_interface name="effort"/>
+        </joint>
+        <joint name="elbow_joint">
+            <command_interface name="position"/>
+            <command_interface name="velocity"/>
+            <state_interface name="position">
+                <param name="initial_value">0</param>
+            </state_interface>
+            <state_interface name="velocity"/>
+            <state_interface name="effort"/>
+        </joint>
+        <joint name="wrist_1_joint">
+            <command_interface name="position"/>
+            <command_interface name="velocity"/>
+            <state_interface name="position">
+                <param name="initial_value">-1.57</param>
+            </state_interface>
+            <state_interface name="velocity"/>
+            <state_interface name="effort"/>
+        </joint>
+        <joint name="wrist_2_joint">
+            <command_interface name="position"/>
+            <command_interface name="velocity"/>
+            <state_interface name="position">
+                <param name="initial_value">0</param>
+            </state_interface>
+            <state_interface name="velocity"/>
+            <state_interface name="effort"/>
+        </joint>
+        <joint name="wrist_3_joint">
+            <command_interface name="position"/>
+            <command_interface name="velocity"/>
+            <state_interface name="position">
+                <param name="initial_value">0</param>
+            </state_interface>
+            <state_interface name="velocity"/>
+            <state_interface name="effort"/>
+        </joint>
+        <!-- Gripper Hardware Interface -->
+      <joint name="robotiq_85_left_knuckle_joint">
+        <command_interface name="position"/>
+        <state_interface name="position">
+          <param name="initial_value">0</param>
+        </state_interface>
+        <state_interface name="velocity"/>
+      </joint>
+      <joint name="robotiq_85_left_inner_knuckle_joint">
+        <param name="mimic">robotiq_85_left_knuckle_joint</param>
+        <param name="offset">0.0</param>
+        <command_interface name="position"/>
+        <state_interface name="position">
+          <param name="initial_value">0</param>
+        </state_interface>
+        <state_interface name="velocity"/>
+      </joint>
+      <joint name="robotiq_85_left_finger_joint">
+        <command_interface name="position"/>
+        <state_interface name="position">
+          <param name="initial_value">0</param>
+        </state_interface>
+        <state_interface name="velocity"/>
+      </joint>
+      <joint name="robotiq_85_left_finger_tip_joint">
+        <param name="mimic">robotiq_85_left_knuckle_joint</param>
+        <param name="multiplier">-1.0</param>
+        <command_interface name="position"/>
+        <state_interface name="position">
+          <param name="initial_value">0</param>
+        </state_interface>
+        <state_interface name="velocity"/>
+      </joint>
+      <joint name="robotiq_85_right_knuckle_joint">
+        <param name="mimic">robotiq_85_left_knuckle_joint</param>
+        <param name="multiplier">1.0</param>
+        <command_interface name="position"/>
+        <state_interface name="position">
+          <param name="initial_value">0</param>
+        </state_interface>
+        <state_interface name="velocity"/>
+      </joint>
+      <joint name="robotiq_85_right_inner_knuckle_joint">
+        <param name="mimic">robotiq_85_left_knuckle_joint</param>
+        <param name="offset">0.0</param>
+        <command_interface name="position"/>
+        <state_interface name="position">
+          <param name="initial_value">0</param>
+        </state_interface>
+        <state_interface name="velocity"/>
+      </joint>
+      <joint name="robotiq_85_right_finger_joint">
+        <command_interface name="position"/>
+        <state_interface name="position">
+          <param name="initial_value">0</param>
+        </state_interface>
+        <state_interface name="velocity"/>
+      </joint>
+      <joint name="robotiq_85_right_finger_tip_joint">
+        <param name="mimic">robotiq_85_left_knuckle_joint</param>
+        <param name="multiplier">-1.0</param>
+        <command_interface name="position"/>
+        <state_interface name="position">
+          <param name="initial_value">0</param>
+        </state_interface>
+        <state_interface name="velocity"/>
+      </joint>
     </ros2_control>
     <!-- Gazebo plugin to parse ros2_control tag and load hardware interface + controller manager -->
